File: kicad/pNC-01/pNC-01.sch (KiCad schematic (older format))
At the start: 5 parts, among them J1 DB25_Female, J2 DB25_Female, J3 DB25_Female

Commit message: fuss with kicad
flarm
Parts:
- removed SW?: SW_SPST_Lamp, symbol Switch:SW_SPST_Lamp
- added 110VAC: AC, symbol power:AC
- added F1: 20A SLOWBLOW, 74, symbol Device:Fuse
- added F2: 500mA FAST, 74, symbol Device:Fuse
- added F3: 2.5A FAST, 74, symbol Device:Fuse
- added F4: 15A SLOWBLOW, 74, symbol Device:Fuse
- added SW?: SW_SPST_Lamp, symbol Switch:SW_SPST_Lamp
Connections:
- net labels added: Earth, LINE, NEUT
- net labels removed: AC
- wire segments 0 -> 2
Changed lines of the file:
@@
 $EndComp
 $Comp
-L power:AC #PWR?
+L power:AC 110VAC
 U 1 1 5CD0CC59
-P 4850 2900
-F 0 "#PWR?" H 4850 2800 50  0001 C CNN
-F 1 "AC" H 4850 3175 50  0000 C CNN
-F 2 "" H 4850 2900 50  0001 C CNN
-F 3 "" H 4850 2900 50  0001 C CNN
-	1    4850 2900
+P 1850 2150
+F 0 "110VAC" H 1955 2284 50  0000 L CNN
+F 1 "AC" H 1955 2193 50  0000 L CNN
+F 2 "" H 1850 2150 50  0001 C CNN
+F 3 "" H 1850 2150 50  0001 C CNN
+	1    1850 2150
 	1    0    0    -1
 $EndComp
@@
 $Comp
 L Switch:SW_SPST_Lamp SW?
-U 1 1 5CD0F8DC
-P 5350 3400
-F 0 "SW?" H 5350 3730 50  0000 C CNN
-F 1 "SW_SPST_Lamp" H 5350 3639 50  0000 C CNN
-F 2 "" H 5350 3700 50  0001 C CNN
-F 3 "~" H 5350 3700 50  0001 C CNN
-	1    5350 3400
+U 1 1 5CD14961
+P 2450 3400
+F 0 "SW?" H 2450 3730 50  0000 C CNN
+F 1 "SW_SPST_Lamp" H 2450 3639 50  0000 C CNN
+F 2 "" H 2450 3700 50  0001 C CNN
+F 3 "~" H 2450 3700 50  0001 C CNN
+	1    2450 3400
 	1    0    0    -1
 $EndComp
+Wire Wire Line
+	2650 3300 2650 3400
+Wire Wire Line
+	2650 3300 2750 3300
+Connection ~ 2650 3300
+$Comp
+L Device:Fuse F1
+U 1 1 5CD16D81
+P 1000 2650
+F 0 "F1" V 902 2696 50  0000 R CNN
+F 1 "20A SLOWBLOW" V 1060 2605 31  0000 C TNN
+F 2 "74" V 930 2650 50  0001 C CNN
+F 3 "~" H 1000 2650 50  0001 C CNN
+	1    1000 2650
+	1    0    0    -1
+$EndComp
+$Comp
+L Device:Fuse F2
+U 1 1 5CD198E1
+P 1500 2650
+F 0 "F2" V 1402 2696 50  0000 R CNN
+F 1 "500mA FAST" V 1560 2605 31  0000 C TNN
+F 2 "74" V 1430 2650 50  0001 C CNN
+F 3 "~" H 1500 2650 50  0001 C CNN
+	1    1500 2650
+	1    0    0    -1
+$EndComp
+$Comp
+L Device:Fuse F3
+U 1 1 5CD1A359
+P 2000 2650
+F 0 "F3" V 1902 2696 50  0000 R CNN
+F 1 "2.5A FAST" V 2060 2605 31  0000 C TNN
+F 2 "74" V 1930 2650 50  0001 C CNN
+F 3 "~" H 2000 2650 50  0001 C CNN
+	1    2000 2650
+	1    0    0    -1
+$EndComp
+$Comp
+L Device:Fuse F4
+U 1 1 5CD1A886
+P 2500 2650
+F 0 "F4" V 2402 2696 50  0000 R CNN
+F 1 "15A SLOWBLOW" V 2560 2605 31  0000 C TNN
+F 2 "74" V 2430 2650 50  0001 C CNN
+F 3 "~" H 2500 2650 50  0001 C CNN
+	1    2500 2650
+	1    0    0    -1
+$EndComp
+$Comp
+L power:Earth #PWR?
+U 1 1 5CD1CAE9
+P 650 2250
+F 0 "#PWR?" H 650 2000 50  0001 C CNN
+F 1 "Earth" H 650 2100 50  0001 C CNN
+F 2 "" H 650 2250 50  0001 C CNN
+F 3 "~" H 650 2250 50  0001 C CNN
+	1    650  2250
+	1    0    0    -1
+$EndComp
+$Comp
+L power:LINE #PWR?
+U 1 1 5CD1DB05
+P 950 2250
+F 0 "#PWR?" H 950 2100 50  0001 C CNN
+F 1 "LINE" H 967 2423 50  0000 C CNN
+F 2 "" H 950 2250 50  0001 C CNN
+F 3 "" H 950 2250 50  0001 C CNN
+	1    950  2250
+	1    0    0    -1
+$EndComp
+$Comp
+L power:NEUT #PWR?
+U 1 1 5CD1EC95
+P 750 2250
+F 0 "#PWR?" H 750 2100 50  0001 C CNN
+F 1 "NEUT" H 767 2423 50  0000 C CNN
+F 2 "" H 750 2250 50  0001 C CNN
+F 3 "" H 750 2250 50  0001 C CNN
+	1    750  2250
+	1    0    0    -1
+$EndComp

Commit message: KICADS
KICADS
Parts:
- removed SW?: SW_SPST_Lamp, symbol Switch:SW_SPST_Lamp
- added Maxon_DCX_01: Motor_DC, symbol Motor:Motor_DC
- added SW1: SW_SPST_PWR_LAMP, symbol encoder_maxon_dcx:SW_SPST_PWD_LAMP
Connections:
- wire segments 2 -> 0
Other:
- moved on the sheet: F1, F2, F3, F4
Changed lines of the file:
@@
 EESchema Schematic File Version 4
+LIBS:pNC-01-cache
 EELAYER 29 0
 EELAYER END
@@
 L power:AC 110VAC
 U 1 1 5CD0CC59
-P 1850 2150
-F 0 "110VAC" H 1955 2284 50  0000 L CNN
-F 1 "AC" H 1955 2193 50  0000 L CNN
-F 2 "" H 1850 2150 50  0001 C CNN
-F 3 "" H 1850 2150 50  0001 C CNN
-	1    1850 2150
+P 2475 3250
+F 0 "110VAC" H 2580 3384 50  0000 L CNN
+F 1 "AC" H 2580 3293 50  0000 L CNN
+F 2 "" H 2475 3250 50  0001 C CNN
+F 3 "" H 2475 3250 50  0001 C CNN
+	1    2475 3250
 	1    0    0    -1
 $EndComp
@@
 $EndComp
 $Comp
-L Switch:SW_SPST_Lamp SW?
-U 1 1 5CD14961
-P 2450 3400
-F 0 "SW?" H 2450 3730 50  0000 C CNN
-F 1 "SW_SPST_Lamp" H 2450 3639 50  0000 C CNN
-F 2 "" H 2450 3700 50  0001 C CNN
-F 3 "~" H 2450 3700 50  0001 C CNN
-	1    2450 3400
-	1    0    0    -1
-$EndComp
-Wire Wire Line
-	2650 3300 2650 3400
-Wire Wire Line
-	2650 3300 2750 3300
-Connection ~ 2650 3300
-$Comp
 L Device:Fuse F1
 U 1 1 5CD16D81
-P 1000 2650
-F 0 "F1" V 902 2696 50  0000 R CNN
-F 1 "20A SLOWBLOW" V 1060 2605 31  0000 C TNN
-F 2 "74" V 930 2650 50  0001 C CNN
-F 3 "~" H 1000 2650 50  0001 C CNN
-	1    1000 2650
+P 1500 4650
+F 0 "F1" V 1402 4696 50  0000 R CNN
+F 1 "20A SLOWBLOW" V 1560 4605 31  0000 C TNN
+F 2 "74" V 1430 4650 50  0001 C CNN
+F 3 "~" H 1500 4650 50  0001 C CNN
+	1    1500 4650
 	1    0    0    -1
 $EndComp
@@
 L Device:Fuse F2
 U 1 1 5CD198E1
-P 1500 2650
-F 0 "F2" V 1402 2696 50  0000 R CNN
-F 1 "500mA FAST" V 1560 2605 31  0000 C TNN
-F 2 "74" V 1430 2650 50  0001 C CNN
-F 3 "~" H 1500 2650 50  0001 C CNN
-	1    1500 2650
+P 2000 4650
+F 0 "F2" V 1902 4696 50  0000 R CNN
+F 1 "500mA FAST" V 2060 4605 31  0000 C TNN
+F 2 "74" V 1930 4650 50  0001 C CNN
+F 3 "~" H 2000 4650 50  0001 C CNN
+	1    2000 4650
 	1    0    0    -1
 $EndComp
@@
 L Device:Fuse F3
 U 1 1 5CD1A359
-P 2000 2650
-F 0 "F3" V 1902 2696 50  0000 R CNN
-F 1 "2.5A FAST" V 2060 2605 31  0000 C TNN
-F 2 "74" V 1930 2650 50  0001 C CNN
-F 3 "~" H 2000 2650 50  0001 C CNN
-	1    2000 2650
+P 2500 4650
+F 0 "F3" V 2402 4696 50  0000 R CNN
+F 1 "2.5A FAST" V 2560 4605 31  0000 C TNN
+F 2 "74" V 2430 4650 50  0001 C CNN
+F 3 "~" H 2500 4650 50  0001 C CNN
+	1    2500 4650
 	1    0    0    -1
 $EndComp
@@
 L Device:Fuse F4
 U 1 1 5CD1A886
-P 2500 2650
-F 0 "F4" V 2402 2696 50  0000 R CNN
-F 1 "15A SLOWBLOW" V 2560 2605 31  0000 C TNN
-F 2 "74" V 2430 2650 50  0001 C CNN
-F 3 "~" H 2500 2650 50  0001 C CNN
-	1    2500 2650
+P 3000 4650
+F 0 "F4" V 2902 4696 50  0000 R CNN
+F 1 "15A SLOWBLOW" V 3060 4605 31  0000 C TNN
+F 2 "74" V 2930 4650 50  0001 C CNN
+F 3 "~" H 3000 4650 50  0001 C CNN
+	1    3000 4650
 	1    0    0    -1
 $EndComp
@@
 L power:Earth #PWR?
 U 1 1 5CD1CAE9
-P 650 2250
-F 0 "#PWR?" H 650 2000 50  0001 C CNN
-F 1 "Earth" H 650 2100 50  0001 C CNN
-F 2 "" H 650 2250 50  0001 C CNN
-F 3 "~" H 650 2250 50  0001 C CNN
-	1    650  2250
+P 1100 4000
+F 0 "#PWR?" H 1100 3750 50  0001 C CNN
+F 1 "Earth" V 1100 3800 50  0000 C CNN
+F 2 "" H 1100 4000 50  0001 C CNN
+F 3 "~" H 1100 4000 50  0001 C CNN
+	1    1100 4000
 	1    0    0    -1
 $EndComp
@@
 L power:LINE #PWR?
 U 1 1 5CD1DB05
-P 950 2250
-F 0 "#PWR?" H 950 2100 50  0001 C CNN
-F 1 "LINE" H 967 2423 50  0000 C CNN
-F 2 "" H 950 2250 50  0001 C CNN
-F 3 "" H 950 2250 50  0001 C CNN
-	1    950  2250
-	1    0    0    -1
+P 1400 4000
+F 0 "#PWR?" H 1400 3850 50  0001 C CNN
+F 1 "LINE" V 1400 4200 50  0000 C CNN
+F 2 "" H 1400 4000 50  0001 C CNN
+F 3 "" H 1400 4000 50  0001 C CNN
+	1    1400 4000
+	-1   0    0    1
 $EndComp
 $Comp
 L power:NEUT #PWR?
 U 1 1 5CD1EC95
-P 750 2250
-F 0 "#PWR?" H 750 2100 50  0001 C CNN
-F 1 "NEUT" H 767 2423 50  0000 C CNN
-F 2 "" H 750 2250 50  0001 C CNN
-F 3 "" H 750 2250 50  0001 C CNN
-	1    750  2250
-	1    0    0    -1
+P 1250 4000
+F 0 "#PWR?" H 1250 3850 50  0001 C CNN
+F 1 "NEUT" V 1250 4200 50  0000 C CNN
+F 2 "" H 1250 4000 50  0001 C CNN
+F 3 "" H 1250 4000 50  0001 C CNN
+	1    1250 4000
+	-1   0    0    1
 $EndComp
+$Comp
+L Motor:Motor_DC Maxon_DCX_01
+U 1 1 5CD8D988
+P 5150 5800
+F 0 "Maxon_DCX_01" V 5445 5750 50  0000 C CNN
+F 1 "Motor_DC" V 5354 5750 50  0000 C CNN
+F 2 "" H 5150 5710 50  0001 C CNN
+F 3 "~" H 5150 5710 50  0001 C CNN
+	1    5150 5800
+	0    -1   -1   0
+$EndComp
+$Comp
+L encoder_maxon_dcx:SW_SPST_PWD_LAMP SW1
+U 1 1 5CD9257B
+P 1950 3100
+F 0 "SW1" V 2050 3250 50  0000 L CNN
+F 1 "SW_SPST_PWR_LAMP" H 2086 3249 50  0001 L CNN
+F 2 "" H 2000 3500 50  0001 C CNN
+F 3 "~" H 2000 3500 50  0001 C CNN
+	1    1950 3100
+	0    -1   -1   0
+$EndComp
+Wire Notes Line
+	1025 4025 1450 4025
+Wire Notes Line
+	1450 4025 1450 4325
+Wire Notes Line
+	1450 4325 1025 4325
+Wire Notes Line
+	1025 4325 1025 4025
 $EndSCHEMATC

Commit message: WIP
WIP
Parts:
- removed 110VAC: AC, symbol power:AC
- K1: renamed from K?; value Fujitsu_FTR-F1A -> OMRON_G7L-2A-BUBJ-CB AC100/120
Connections:
- net LINE: now also F1.2, F2.2
- net NEUT: now also K1.2, K1.4, SW1.3 (LAMP_NEUT)
- net at K1.5: now also SW1.2 (OUT)
- net at K1.7: now also F1.1
- net at F2.1: now also SW1.1 (IN)
Other:
- moved on the sheet: F1, F2, F3, F4, K1, SW1
Changed lines of the file:
@@
 $EndComp
 $Comp
-L power:AC 110VAC
-U 1 1 5CD0CC59
-P 2475 3250
-F 0 "110VAC" H 2580 3384 50  0000 L CNN
-F 1 "AC" H 2580 3293 50  0000 L CNN
-F 2 "" H 2475 3250 50  0001 C CNN
-F 3 "" H 2475 3250 50  0001 C CNN
-	1    2475 3250
-	1    0    0    -1
-$EndComp
-$Comp
-L Relay:Fujitsu_FTR-F1A K?
+L Relay:Fujitsu_FTR-F1A K1
 U 1 1 5CD0D6B4
-P 6200 2700
-F 0 "K?" H 6200 3217 50  0000 C CNN
-F 1 "Fujitsu_FTR-F1A" H 6200 3126 50  0000 C CNN
-F 2 "Relay_THT:Relay_DPST_Fujitsu_FTR-F1A" H 6200 2300 50  0001 C CNN
-F 3 "https://www.fujitsu.com/downloads/MICRO/fcai/relays/ftr-f1.pdf" H 6250 3250 50  0001 C CNN
-	1    6200 2700
+P 2725 3675
+F 0 "K1" H 2725 4192 50  0000 C CNN
+F 1 "OMRON_G7L-2A-BUBJ-CB AC100/120" H 2725 4101 50  0000 C CNN
+F 2 "Relay_THT:Relay_DPST_Fujitsu_FTR-F1A" H 2725 3275 50  0001 C CNN
+F 3 "https://www.fujitsu.com/downloads/MICRO/fcai/relays/ftr-f1.pdf" H 2775 4225 50  0001 C CNN
+	1    2725 3675
 	1    0    0    -1
 $EndComp
@@
 L Device:Fuse F1
 U 1 1 5CD16D81
-P 1500 4650
-F 0 "F1" V 1402 4696 50  0000 R CNN
-F 1 "20A SLOWBLOW" V 1560 4605 31  0000 C TNN
-F 2 "74" V 1430 4650 50  0001 C CNN
-F 3 "~" H 1500 4650 50  0001 C CNN
-	1    1500 4650
-	1    0    0    -1
+P 1850 3675
+F 0 "F1" V 1752 3721 50  0000 R CNN
+F 1 "20A SLOWBLOW" V 1910 3630 31  0000 C TNN
+F 2 "74" V 1780 3675 50  0001 C CNN
+F 3 "~" H 1850 3675 50  0001 C CNN
+	1    1850 3675
+	0    1    1    0
 $EndComp
 $Comp
 L Device:Fuse F2
 U 1 1 5CD198E1
-P 2000 4650
-F 0 "F2" V 1902 4696 50  0000 R CNN
-F 1 "500mA FAST" V 2060 4605 31  0000 C TNN
-F 2 "74" V 1930 4650 50  0001 C CNN
-F 3 "~" H 2000 4650 50  0001 C CNN
-	1    2000 4650
+P 1150 3125
+F 0 "F2" V 1052 3171 50  0000 R CNN
+F 1 "500mA FAST" V 1210 3080 31  0000 C TNN
+F 2 "74" V 1080 3125 50  0001 C CNN
+F 3 "~" H 1150 3125 50  0001 C CNN
+	1    1150 3125
 	1    0    0    -1
 $EndComp
@@
 L Device:Fuse F3
 U 1 1 5CD1A359
-P 2500 4650
-F 0 "F3" V 2402 4696 50  0000 R CNN
-F 1 "2.5A FAST" V 2560 4605 31  0000 C TNN
-F 2 "74" V 2430 4650 50  0001 C CNN
-F 3 "~" H 2500 4650 50  0001 C CNN
-	1    2500 4650
-	1    0    0    -1
+P 3900 3750
+F 0 "F3" V 3802 3796 50  0000 R CNN
+F 1 "2.5A FAST" V 3960 3705 31  0000 C TNN
+F 2 "74" V 3830 3750 50  0001 C CNN
+F 3 "~" H 3900 3750 50  0001 C CNN
+	1    3900 3750
+	0    1    1    0
 $EndComp
 $Comp
 L Device:Fuse F4
 U 1 1 5CD1A886
-P 3000 4650
-F 0 "F4" V 2902 4696 50  0000 R CNN
-F 1 "15A SLOWBLOW" V 3060 4605 31  0000 C TNN
-F 2 "74" V 2930 4650 50  0001 C CNN
-F 3 "~" H 3000 4650 50  0001 C CNN
-	1    3000 4650
-	1    0    0    -1
+P 3900 4000
+F 0 "F4" V 3802 4046 50  0000 R CNN
+F 1 "15A SLOWBLOW" V 3960 3955 31  0000 C TNN
+F 2 "74" V 3830 4000 50  0001 C CNN
+F 3 "~" H 3900 4000 50  0001 C CNN
+	1    3900 4000
+	0    1    1    0
 $EndComp
 $Comp
@@
 L power:LINE #PWR?
 U 1 1 5CD1DB05
-P 1400 4000
-F 0 "#PWR?" H 1400 3850 50  0001 C CNN
-F 1 "LINE" V 1400 4200 50  0000 C CNN
-F 2 "" H 1400 4000 50  0001 C CNN
-F 3 "" H 1400 4000 50  0001 C CNN
-	1    1400 4000
+P 1250 4000
+F 0 "#PWR?" H 1250 3850 50  0001 C CNN
+F 1 "LINE" V 1250 4225 50  0000 C CNN
+F 2 "" H 1250 4000 50  0001 C CNN
+F 3 "" H 1250 4000 50  0001 C CNN
+	1    1250 4000
 	-1   0    0    1
 $EndComp
@@
 L power:NEUT #PWR?
 U 1 1 5CD1EC95
-P 1250 4000
-F 0 "#PWR?" H 1250 3850 50  0001 C CNN
-F 1 "NEUT" V 1250 4200 50  0000 C CNN
-F 2 "" H 1250 4000 50  0001 C CNN
-F 3 "" H 1250 4000 50  0001 C CNN
-	1    1250 4000
+P 1400 4000
+F 0 "#PWR?" H 1400 3850 50  0001 C CNN
+F 1 "NEUT" V 1400 4200 50  0000 C CNN
+F 2 "" H 1400 4000 50  0001 C CNN
+F 3 "" H 1400 4000 50  0001 C CNN
+	1    1400 4000
 	-1   0    0    1
 $EndComp
@@
 L encoder_maxon_dcx:SW_SPST_PWD_LAMP SW1
 U 1 1 5CD9257B
-P 1950 3100
-F 0 "SW1" V 2050 3250 50  0000 L CNN
-F 1 "SW_SPST_PWR_LAMP" H 2086 3249 50  0001 L CNN
-F 2 "" H 2000 3500 50  0001 C CNN
-F 3 "~" H 2000 3500 50  0001 C CNN
-	1    1950 3100
+P 1450 2675
+F 0 "SW1" V 1550 2825 50  0000 L CNN
+F 1 "SW_SPST_PWR_LAMP" H 1586 2824 50  0001 L CNN
+F 2 "" H 1500 3075 50  0001 C CNN
+F 3 "~" H 1500 3075 50  0001 C CNN
+	1    1450 2675
 	0    -1   -1   0
 $EndComp
@@
 Wire Notes Line
 	1025 4325 1025 4025
+Wire Wire Line
+	1250 3425 1700 3675
+Wire Wire Line
+	1250 3425 1150 3275
+Wire Wire Line
+	1250 3425 1250 4000
+Connection ~ 1250 3425
+Wire Wire Line
+	1150 2875 1150 2975
+Wire Wire Line
+	1350 2875 1400 3225
+Wire Wire Line
+	1400 3225 1400 3925
+Wire Wire Line
+	1250 2875 1250 2975
+Wire Wire Line
+	1250 2975 1950 2975
+Wire Wire Line
+	1950 2975 1950 3475
+Wire Wire Line
+	1950 3475 2425 3475
+Wire Wire Line
+	2000 3675 2425 3675
+Wire Wire Line
+	1400 3925 2425 3925
+Wire Wire Line
+	2425 3925 2425 3875
+Connection ~ 1400 3925
+Wire Wire Line
+	1400 3925 1400 4000
+$Comp
+L power:NEUT #PWR?
+U 1 1 5CDB68B7
+P 3200 3475
+F 0 "#PWR?" H 3200 3325 50  0001 C CNN
+F 1 "NEUT" V 3217 3603 50  0000 L CNN
+F 2 "" H 3200 3475 50  0001 C CNN
+F 3 "" H 3200 3475 50  0001 C CNN
+	1    3200 3475
+	0    1    1    0
+$EndComp
+Wire Wire Line
+	3025 3475 3200 3475
 $EndSCHEMATC

Commit message: lolhowdoesicircuiting?
Parts:
- added J?: Encoder_Maxon_DCX, symbol encoder_maxon_dcx:Encoder_Maxon_DCX
Connections:
- net at K1.8: now also F3.2, F4.2
Other:
- moved on the sheet: F3, F4
Changed lines of the file:
@@
 U 1 1 5CD0D6B4
 P 2725 3675
-F 0 "K1" H 2725 4192 50  0000 C CNN
-F 1 "OMRON_G7L-2A-BUBJ-CB AC100/120" H 2725 4101 50  0000 C CNN
+F 0 "K1" H 2725 4125 50  0000 C CNN
+F 1 "OMRON_G7L-2A-BUBJ-CB AC100/120" H 2725 4075 20  0000 C CNN
 F 2 "Relay_THT:Relay_DPST_Fujitsu_FTR-F1A" H 2725 3275 50  0001 C CNN
 F 3 "https://www.fujitsu.com/downloads/MICRO/fcai/relays/ftr-f1.pdf" H 2775 4225 50  0001 C CNN
@@
 L Device:Fuse F3
 U 1 1 5CD1A359
-P 3900 3750
-F 0 "F3" V 3802 3796 50  0000 R CNN
-F 1 "2.5A FAST" V 3960 3705 31  0000 C TNN
-F 2 "74" V 3830 3750 50  0001 C CNN
-F 3 "~" H 3900 3750 50  0001 C CNN
-	1    3900 3750
+P 3900 3500
+F 0 "F3" V 3825 3550 50  0000 R CNN
+F 1 "2.5A FAST" V 3950 3500 25  0000 C TNN
+F 2 "74" V 3830 3500 50  0001 C CNN
+F 3 "~" H 3900 3500 50  0001 C CNN
+	1    3900 3500
 	0    1    1    0
 $EndComp
@@
 L Device:Fuse F4
 U 1 1 5CD1A886
-P 3900 4000
-F 0 "F4" V 3802 4046 50  0000 R CNN
-F 1 "15A SLOWBLOW" V 3960 3955 31  0000 C TNN
-F 2 "74" V 3830 4000 50  0001 C CNN
-F 3 "~" H 3900 4000 50  0001 C CNN
-	1    3900 4000
+P 3900 3825
+F 0 "F4" V 3825 3875 50  0000 R CNN
+F 1 "15A SLOWBLOW" V 3950 3825 25  0000 C TNN
+F 2 "74" V 3830 3825 50  0001 C CNN
+F 3 "~" H 3900 3825 50  0001 C CNN
+	1    3900 3825
 	0    1    1    0
 $EndComp
@@
 	1350 2875 1400 3225
 Wire Wire Line
-	1400 3225 1400 3925
+	1400 3225 1400 3875
 Wire Wire Line
 	1250 2875 1250 2975
@@
 	2000 3675 2425 3675
 Wire Wire Line
-	1400 3925 2425 3925
+	1400 3875 2425 3875
+Connection ~ 1400 3875
 Wire Wire Line
-	2425 3925 2425 3875
-Connection ~ 1400 3925
-Wire Wire Line
-	1400 3925 1400 4000
+	1400 3875 1400 4000
 $Comp
 L power:NEUT #PWR?
@@
 P 3200 3475
 F 0 "#PWR?" H 3200 3325 50  0001 C CNN
-F 1 "NEUT" V 3217 3603 50  0000 L CNN
+F 1 "NEUT" V 3200 3575 25  0000 L CNN
 F 2 "" H 3200 3475 50  0001 C CNN
 F 3 "" H 3200 3475 50  0001 C CNN
@@
 Wire Wire Line
 	3025 3475 3200 3475
+Wire Wire Line
+	3025 3675 3575 3675
+Wire Wire Line
+	3575 3675 3750 3500
+Wire Wire Line
+	3575 3675 3750 3825
+Connection ~ 3575 3675
+$Comp
+L encoder_maxon_dcx:Encoder_Maxon_DCX J?
+U 1 1 5CDBCA1B
+P 6350 5950
+F 0 "J?" V 6354 6230 50  0000 L CNN
+F 1 "Encoder_Maxon_DCX" V 6445 6230 50  0000 L CNN
+F 2 "" H 6350 5950 50  0001 C CNN
+F 3 "~" H 6350 5950 50  0001 C CNN
+	1    6350 5950
+	0    1    1    0
+$EndComp
 $EndSCHEMATC
